File: iobbq_solar_charger.sch (EAGLE design)
At the start: 29 parts, among them X1 TE_RUUVULIITIN2, X2 TE_RUUVULIITIN2, X3 TE_RUUVULIITIN2, X4 TE_RUUVULIITIN2

Commit message: update values
Parts:
- added U$2: DAFUG, dafug:DAFUG
- C2: value CAP0805 -> 4µ7
- C4: value CAP0805 -> 2µ2 50V
- H1: value (none) -> GRN
- H2: value (none) -> RED
- L1: value (none) -> WE-PD-7447779122
- R1, R2, R8: value RES0603 -> 100k
- R10, R9: value RES1206 -> 2k15
- R11: value RES1206 -> 0.1R 1206
- R3: value RES0603 -> NCP18XH103
- R4: value RES0603 -> 910R
- R5: value RES0603 -> 174k
- R6: value RES0603 -> 1M
- R7: value RES0603 -> 309k
- V1, V5: value (none) -> MBRS340
- V4: value BZX84CSMD -> BZX84C 6V2
- X1, X2, X3, X4: value TE_RUUVULIITIN2 -> TE 282837-2; device OMAT_IC:TE_RUUVULIITIN2 -> OMAT_IC:TE_RUUVILIITIN2
Other:
- note added: "DO NOT ASSEMBLY LEDS IF SIGNALS ARE USED EXTERNALLY WITH LOWER VOLTAGE"
- note added: "NTC 10k 0603"
- note added: "SOLAR PANEL BATTERY CHARGER KIMMOLI 2015"
- note removed: "NTC"
- moved on the sheet: H1, H2, R10, R9, V1, X2
